File: 8Bit Computer ver2.0/Kicad/Computer/Computer.kicad_pcb (KiCad board)
At the start: 4 copper layers, 633.2 x 616.8 mm, 666 parts, among them IC1 MP2338GTL-Z, IC10 SN74LVC1G14DBVR, IC100 SN74ABT574ADWR, IC101 SN74LVC1G14DBVR, IC102 SN74AHC86DR, IC103 SN74AHC74DR, IC104 SN74ABT574ADWR, IC105 SN74LVC1G14DBVR, IC106 SN74AHC08DR, IC107 SN74AHC08DR, IC108 SN74AHC74DR, IC109 SN74ABT574ADWR, IC11 SN74LVC1G14DBVR, IC110 SN74LVC1G14DBVR, IC111 SN74AHC14DR, IC112 SN74AHC14DR, IC113 SN74AHC74DR, IC114 SN74ABT574ADWR, IC115 SN74LVC1G14DBVR, IC116 SN74AHC32DR, IC117 SN74AHC32DR, IC118 SN74AHC74DR, IC119 SN74ABT574ADWR, IC12 SN74LVC1G14DBVR, IC120 SN74LVC1G14DBVR, IC121 SN74AHC86DR, IC122 SN74AHC86DR, IC123 SN74AHC74DR, IC124 SN74ABT574ADWR, IC125 SN74LVC1G14DBVR, IC126 SN74AHC32DR, IC127 SN74HCS4075DR, IC128 SN74AHC08DR, IC129 SN74AHC74DR, IC13 SN74LVC1G14DBVR, IC130 SN74AHC74DR, IC131 SN74AHC74DR, IC132 SN74AHC08DR, IC133 SN74ABT574ADWR, IC134 SN74ABT245BDWR, IC135 SN74LVC1G32DBVR, IC136 SN74LVC1G14DBVR, IC137 SN74LVC1G14DBVR, IC138 SN74AHC74DR, IC139 SN74F283D, IC14 SN74LVC1G14DBVR, IC140 SN74F283D, IC141 SN74F283D, IC142 SN74LVC1G86DBVR, IC143 SN74ABT574ADWR, IC144 SN74ABT574ADWR, IC145 SN74LVC1G14DBVR, IC146 SN74LVC1G14DBVR, IC147 SN74HC682N, IC148 SN74AHC08DR, IC149 SN74HCS4075DR, IC15 SN74LVC1G14DBVR, IC150 SN74AHC74DR, IC151 SN74LVC1G14DBVR, IC152 SN74LVC1G14DBVR, IC153 SN74LVC1G08DBVR, IC154 SN74ABT574ADWR, IC155 SN74F521DWR, IC156 SN74F521DWR, IC157 SN74LVC1G14DBVR, IC158 SN74LVC1G14DBVR, IC159 SN74LVC1G14DBVR, IC16 SN74LVC1G14DBVR, IC160 SN74LVC1G08DBVR, IC161 SN74LVC1G32DBVR, IC162 SN74HCS4075DR, IC163 SN74LVC1G32DBVR, IC164 SN74LVC1G14DBVR, IC165 CY74FCT163CTSOC, IC166 CY74FCT163CTSOC, IC167 CY74FCT163CTSOC, IC168 CY74FCT163CTSOC, IC169 SN74LVC1G14DBVR, IC17 SN74LVC1G14DBVR, IC170 SN74LVC1G32DBVR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

Commit message: tag der offenen Tür
Parts:
- moved IC225 21.0 mm to (702.0, 468.9)
- moved IC231 21.0 mm to (727.9, 468.9)
- moved IC234 21.0 mm to (702.0, 483.4)
- moved IC228 21.0 mm to (685.2, 497.6)
- moved IC229 21.0 mm to (685.2, 502.2)
- moved IC233 21.0 mm to (692.1, 495.9)
- moved IC224 21.0 mm to (689.1, 468.9)
- moved IC226 21.0 mm to (715.0, 468.9)
- moved IC227 21.0 mm to (685.2, 493.0)
- moved IC230 21.0 mm to (685.2, 506.8)
- moved IC232 21.0 mm to (689.1, 483.4)
- moved IC235 21.0 mm to (715.0, 483.4)
Routing:
- net /GNDM: track 185.3 -> 186.7 mm, vias 154 -> 155
Changed lines of the file:
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@@
 	(footprint "Samacsys:SOT95P280X145-5N"
 		(layer "F.Cu")
-		(at 703.535 482.67)
+		(at 685.225 493.02)
 		(descr "DBV (R-PDSO-G5)")
 		(tags "Integrated Circuit")
@@
 		(model "${KIPRJMOD}/Samacsys.3dshapes/2MS1T2B3M2QES.stp"
 			(offset
-				(xyz 0 2.539999924 2.219999995)
+				(xyz 0 2.54 0)
 			)
 			(scale
@@
 			)
 			(rotate
-				(xyz -90 0 -180)
+				(xyz -90 -0 -180)
 			)
 		)
@@
 	(footprint "Samacsys:SOIC127P1030X265-20N"
 		(layer "F.Cu")
-		(at 733.285 473.095)
+		(at 714.975 483.445)
 		(descr "DW0020A")
 		(tags "Integrated Circuit")
@@
 	(footprint "Samacsys:SOIC127P1030X265-20N"
 		(layer "F.Cu")
-		(at 720.335 473.095)
+		(at 702.025 483.445)
 		(descr "DW0020A")
 		(tags "Integrated Circuit")
@@
 	(footprint "Samacsys:SOT95P280X145-5N"
 		(layer "F.Cu")
-		(at 703.535 487.27)
+		(at 685.225 497.62)
 		(descr "DBV (R-PDSO-G5)")
 		(tags "Integrated Circuit")
@@
 	(footprint "Samacsys:SOT95P280X145-5N"
 		(layer "F.Cu")
-		(at 703.535 496.47)
+		(at 685.225 506.82)
 		(descr "DBV (R-PDSO-G5)")
 		(tags "Integrated Circuit")
@@
 	(footprint "Samacsys:SOIC127P1030X265-20N"
 		(layer "F.Cu")
-		(at 707.385 473.095)
+		(at 689.075 483.445)
 		(descr "DW0020A")
 		(tags "Integrated Circuit")
@@
 	(footprint "Samacsys:SOIC127P600X175-14N"
 		(layer "F.Cu")
-		(at 710.41 485.52)
+		(at 692.1 495.87)
 		(descr "D (R-PDSO-G14)")
 		(tags "Integrated Circuit")
@@
 	(footprint "Samacsys:SOIC127P1030X265-20N"
 		(layer "F.Cu")
-		(at 720.335 458.545)
+		(at 702.025 468.895)
 		(descr "DW0020A")
 		(tags "Integrated Circuit")
@@
 		(model "SN74HC682N.stp"
 			(offset
-				(xyz -3.809999886 11.43000013 2.499999962)
+				(xyz 0 0 2.5)
 			)
 			(scale
@@
 			)
 			(rotate
-				(xyz -90 0 0)
+				(xyz -90 -0 -0)
 			)
 		)
@@
 	(footprint "Samacsys:SOIC127P1030X265-20N"
 		(layer "F.Cu")
-		(at 733.285 458.545)
+		(at 714.975 468.895)
 		(descr "DW0020A")
 		(tags "Integrated Circuit")
@@
 	(footprint "Samacsys:SOIC127P1030X265-20N"
 		(layer "F.Cu")
-		(at 746.235 458.545)
+		(at 727.925 468.895)
 		(descr "DW0020A")
 		(tags "Integrated Circuit")
@@
 	(footprint "Samacsys:SOT95P280X145-5N"
 		(layer "F.Cu")
-		(at 703.535 491.87)
+		(at 685.225 502.22)
 		(descr "DBV (R-PDSO-G5)")
 		(tags "Integrated Circuit")
@@
 	(footprint "Samacsys:SOIC127P1030X265-20N"
 		(layer "F.Cu")
-		(at 707.385 458.545)
+		(at 689.075 468.895)
 		(descr "DW0020A")
 		(tags "Integrated Circuit")
@@
 		(net 27)
 	)
+	(gr_line
+		(start 354.25 24.25)
+		(end 354.25 23)
+		(stroke
+			(width 0.1)
+			(type default)
+		)
+		(layer "F.SilkS")
+	)
+	(gr_line
+		(start 358.75 23)
+		(end 358.75 24.25)
+		(stroke
+			(width 0.1)
+			(type default)
+		)
+		(layer "F.SilkS")
+	)
+	(gr_line
+		(start 362.25 73)
+		(end 362.25 74)
+		(stroke
+			(width 0.1)
+			(type default)
+		)
+		(layer "F.SilkS")
+	)
+	(gr_line
+		(start 357.25 74)
+		(end 357.25 73)
+		(stroke
+			(width 0.1)
+			(type default)
+		)
+		(layer "F.SilkS")
+	)
+	(gr_line
+		(start 354.25 23)
+		(end 358.75 23)
+		(stroke
+			(width 0.1)
+			(type default)
+		)
+		(layer "F.SilkS")
+	)
+	(gr_line
+		(start 357.25 73)
+		(end 362.25 73)
+		(stroke
+			(width 0.1)
+			(type default)
+		)
+		(layer "F.SilkS")
+	)
 	(gr_rect
 		(start 168.205128 178.601282)
@@
 	)
 	(segment
+		(start 361.2 54.95)
+		(end 361.5 55.25)
+		(width 0.2)
+		(layer "F.Cu")
+		(net 6)
+	)
+	(segment
 		(start 366.4 50.72)
 		(end 369.28 50.72)
@@
 	)
 	(segment
+		(start 360.2 54.95)
+		(end 361.2 54.95)
+		(width 0.2)
+		(layer "F.Cu")
+		(net 6)
+	)
+	(segment
 		(start 430.95 61.25)
 		(end 431.25 60.95)
@@
 		(size 0.5)
 		(drill 0.3)
+		(layers "F.Cu" "B.Cu")
+		(net 6)
+	)
+	(via
+		(at 361.5 55.25)
+		(size 0.5)
+		(drill 0.3)
