File: 8Bit Computer ver2.0/Kicad/Computer/Computer.kicad_pcb (KiCad board)
At the start: 4 copper layers, 633.2 x 616.8 mm, 666 parts, among them IC1 MP2338GTL-Z, IC10 SN74LVC1G14DBVR, IC100 SN74ABT574ADWR, IC101 SN74LVC1G14DBVR, IC102 SN74AHC86DR, IC103 SN74AHC74DR, IC104 SN74ABT574ADWR, IC105 SN74LVC1G14DBVR, IC106 SN74AHC08DR, IC107 SN74AHC08DR, IC108 SN74AHC74DR, IC109 SN74ABT574ADWR, IC11 SN74LVC1G14DBVR, IC110 SN74LVC1G14DBVR, IC111 SN74AHC14DR, IC112 SN74AHC14DR, IC113 SN74AHC74DR, IC114 SN74ABT574ADWR, IC115 SN74LVC1G14DBVR, IC116 SN74AHC32DR, IC117 SN74AHC32DR, IC118 SN74AHC74DR, IC119 SN74ABT574ADWR, IC12 SN74LVC1G14DBVR, IC120 SN74LVC1G14DBVR, IC121 SN74AHC86DR, IC122 SN74AHC86DR, IC123 SN74AHC74DR, IC124 SN74ABT574ADWR, IC125 SN74LVC1G14DBVR, IC126 SN74AHC32DR, IC127 SN74HCS4075DR, IC128 SN74AHC08DR, IC129 SN74AHC74DR, IC13 SN74LVC1G14DBVR, IC130 SN74AHC74DR, IC131 SN74AHC74DR, IC132 SN74AHC08DR, IC133 SN74ABT574ADWR, IC134 SN74ABT245BDWR, IC135 SN74LVC1G32DBVR, IC136 SN74LVC1G14DBVR, IC137 SN74LVC1G14DBVR, IC138 SN74AHC74DR, IC139 SN74F283D, IC14 SN74LVC1G14DBVR, IC140 SN74F283D, IC141 SN74F283D, IC142 SN74LVC1G86DBVR, IC143 SN74ABT574ADWR, IC144 SN74ABT574ADWR, IC145 SN74LVC1G14DBVR, IC146 SN74LVC1G14DBVR, IC147 SN74HC682N, IC148 SN74AHC08DR, IC149 SN74HCS4075DR, IC15 SN74LVC1G14DBVR, IC150 SN74AHC74DR, IC151 SN74LVC1G14DBVR, IC152 SN74LVC1G14DBVR, IC153 SN74LVC1G08DBVR, IC154 SN74ABT574ADWR, IC155 SN74F521DWR, IC156 SN74F521DWR, IC157 SN74LVC1G14DBVR, IC158 SN74LVC1G14DBVR, IC159 SN74LVC1G14DBVR, IC16 SN74LVC1G14DBVR, IC160 SN74LVC1G08DBVR, IC161 SN74LVC1G32DBVR, IC162 SN74HCS4075DR, IC163 SN74LVC1G32DBVR, IC164 SN74LVC1G14DBVR, IC165 CY74FCT163CTSOC, IC166 CY74FCT163CTSOC, IC167 CY74FCT163CTSOC, IC168 CY74FCT163CTSOC, IC169 SN74LVC1G14DBVR, IC17 SN74LVC1G14DBVR, IC170 SN74LVC1G32DBVR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

Commit message: Kicad
added the Programme Counter und Dat to adr module
Parts:
- added C243: 27pF, Capacitor_SMD:C_1206_3216Metric_Pad1.33x1.80mm_HandSolder, F.Cu at (692.8, 318.1)
- added C244: 100nF, Capacitor_SMD:C_1206_3216Metric_Pad1.33x1.80mm_HandSolder, F.Cu at (686.4, 323.6)
- added C245: 27pF, Capacitor_SMD:C_1206_3216Metric_Pad1.33x1.80mm_HandSolder, F.Cu at (686.2, 318.1)
- added C246: 100nF, Capacitor_SMD:C_1206_3216Metric_Pad1.33x1.80mm_HandSolder, F.Cu at (672.1, 294.4)
- added C247: 100nF, Capacitor_SMD:C_1206_3216Metric_Pad1.33x1.80mm_HandSolder, F.Cu at (678.3, 325.1)
- added C248: 100nF, Capacitor_SMD:C_1206_3216Metric_Pad1.33x1.80mm_HandSolder, F.Cu at (687.4, 283.8)
- added C249: 10nF, Capacitor_SMD:C_1206_3216Metric_Pad1.33x1.80mm_HandSolder, F.Cu at (692.1, 291.9)
- added C250: 4.7uF, Capacitor_SMD:C_1206_3216Metric_Pad1.33x1.80mm_HandSolder, F.Cu at (696.0, 290.1)
- added C251: 100nF, Capacitor_SMD:C_1206_3216Metric_Pad1.33x1.80mm_HandSolder, F.Cu at (664.6, 285.3)
- added C252: 100nF, Capacitor_SMD:C_1206_3216Metric_Pad1.33x1.80mm_HandSolder, F.Cu at (676.6, 285.3)
- added C253: 100nF, Capacitor_SMD:C_1206_3216Metric_Pad1.33x1.80mm_HandSolder, F.Cu at (651.2, 285.3)
- added C254: 100nF, Capacitor_SMD:C_1206_3216Metric_Pad1.33x1.80mm_HandSolder, F.Cu at (664.0, 309.9)
- added C255: 100nF, Capacitor_SMD:C_1206_3216Metric_Pad1.33x1.80mm_HandSolder, F.Cu at (629.1, 356.4)
- added C256: 100nF, Capacitor_SMD:C_1206_3216Metric_Pad1.33x1.80mm_HandSolder, F.Cu at (640.6, 356.4)
- added C257: 100nF, Capacitor_SMD:C_1206_3216Metric_Pad1.33x1.80mm_HandSolder, F.Cu at (628.8, 421.7)
- added C258: 100nF, Capacitor_SMD:C_1206_3216Metric_Pad1.33x1.80mm_HandSolder, F.Cu at (652.4, 356.4)
- added C259: 100nF, Capacitor_SMD:C_1206_3216Metric_Pad1.33x1.80mm_HandSolder, F.Cu at (664.2, 356.3)
- added C260: 100nF, Capacitor_SMD:C_1206_3216Metric_Pad1.33x1.80mm_HandSolder, F.Cu at (643.0, 421.8)
- added C261: 100nF, Capacitor_SMD:C_1206_3216Metric_Pad1.33x1.80mm_HandSolder, F.Cu at (635.7, 377.4)
- added C262: 100nF, Capacitor_SMD:C_1206_3216Metric_Pad1.33x1.80mm_HandSolder, F.Cu at (650.4, 377.4)
- added C263: 100nF, Capacitor_SMD:C_1206_3216Metric_Pad1.33x1.80mm_HandSolder, F.Cu at (657.7, 421.9)
- added C264: 100nF, Capacitor_SMD:C_1206_3216Metric_Pad1.33x1.80mm_HandSolder, F.Cu at (635.9, 393.9)
- added C265: 100nF, Capacitor_SMD:C_1206_3216Metric_Pad1.33x1.80mm_HandSolder, F.Cu at (650.3, 393.9)
- added C266: 100nF, Capacitor_SMD:C_1206_3216Metric_Pad1.33x1.80mm_HandSolder, F.Cu at (671.9, 421.7)
- added C267: 100nF, Capacitor_SMD:C_1206_3216Metric_Pad1.33x1.80mm_HandSolder, F.Cu at (659.0, 405.2)
- added C268: 100nF, Capacitor_SMD:C_1206_3216Metric_Pad1.33x1.80mm_HandSolder, F.Cu at (671.5, 405.6)
- added C269: 100nF, Capacitor_SMD:C_1206_3216Metric_Pad1.33x1.80mm_HandSolder, F.Cu at (686.5, 421.7)
- added C270: 100nF, Capacitor_SMD:C_1206_3216Metric_Pad1.33x1.80mm_HandSolder, F.Cu at (686.5, 352.9)
- added C271: 100nF, Capacitor_SMD:C_1206_3216Metric_Pad1.33x1.80mm_HandSolder, F.Cu at (677.1, 356.1)
- added C272: 100nF, Capacitor_SMD:C_1206_3216Metric_Pad1.33x1.80mm_HandSolder, F.Cu at (632.8, 417.9)
- added C273: 100nF, Capacitor_SMD:C_1206_3216Metric_Pad1.33x1.80mm_HandSolder, F.Cu at (681.6, 371.7)
- added C274: 100nF, Capacitor_SMD:C_1206_3216Metric_Pad1.33x1.80mm_HandSolder, F.Cu at (679.9, 362.8)
- added C275: 100nF, Capacitor_SMD:C_1206_3216Metric_Pad1.33x1.80mm_HandSolder, F.Cu at (646.8, 417.7)
- added C276: 100nF, Capacitor_SMD:C_1206_3216Metric_Pad1.33x1.80mm_HandSolder, F.Cu at (673.8, 343.6)
- added C277: 100nF, Capacitor_SMD:C_1206_3216Metric_Pad1.33x1.80mm_HandSolder, F.Cu at (692.1, 364.0)
- added C278: 100nF, Capacitor_SMD:C_1206_3216Metric_Pad1.33x1.80mm_HandSolder, F.Cu at (661.5, 417.8)
- added C279: 100nF, Capacitor_SMD:C_1206_3216Metric_Pad1.33x1.80mm_HandSolder, F.Cu at (675.8, 417.9)
- added C280: 100nF, Capacitor_SMD:C_1206_3216Metric_Pad1.33x1.80mm_HandSolder, F.Cu at (690.3, 417.9)
- added C281: 100nF, Capacitor_SMD:C_1206_3216Metric_Pad1.33x1.80mm_HandSolder, F.Cu at (672.3, 397.1)
- added C282: 100nF, Capacitor_SMD:C_1206_3216Metric_Pad1.33x1.80mm_HandSolder, F.Cu at (673.1, 389.2)
- added C283: 100nF, Capacitor_SMD:C_1206_3216Metric_Pad1.33x1.80mm_HandSolder, F.Cu at (660.7, 303.4)
- added IC266: SN74LVC1GU04DCKR, Samacsys:SOT65P210X110-5N, F.Cu at (685.7, 320.8)
- added IC267: TMUX1309DYYR, Samacsys:SOP50P326X110-16N, F.Cu at (669.0, 298.1)
- added IC268: SN74LVC1G14DBVR, Samacsys:SOT95P280X145-5N, F.Cu at (679.0, 321.7)
- added IC269: LM555CMX_NOPB, Samacsys:SOIC127P600X175-8N, F.Cu at (686.9, 287.9)
- added IC270: SN74AHC74DR, Samacsys:SOIC127P600X175-14N, F.Cu at (670.0, 308.6)
- added R63: 1M, Resistor_SMD:R_1206_3216Metric_Pad1.30x1.75mm_HandSolder, F.Cu at (682.3, 321.9)
- added R64: 330, Resistor_SMD:R_1206_3216Metric_Pad1.30x1.75mm_HandSolder, F.Cu at (681.0, 318.1)
- added R65: 100, Resistor_SMD:R_1206_3216Metric_Pad1.30x1.75mm_HandSolder, F.Cu at (692.4, 285.1)
- added R66: 1M, Resistor_SMD:R_1206_3216Metric_Pad1.30x1.75mm_HandSolder, F.Cu at (697.7, 284.1)
- added R67: 1500, Resistor_SMD:R_1206_3216Metric_Pad1.30x1.75mm_HandSolder, F.Cu at (695.2, 284.2)
- added R68: 4.7k, Resistor_SMD:R_1206_3216Metric_Pad1.30x1.75mm_HandSolder, F.Cu at (663.1, 280.3)
- added R69: 4.7k, Resistor_SMD:R_1206_3216Metric_Pad1.30x1.75mm_HandSolder, F.Cu at (675.1, 280.3)
- added R70: 4.7k, Resistor_SMD:R_1206_3216Metric_Pad1.30x1.75mm_HandSolder, F.Cu at (649.8, 280.3)
- added R71: 4.7k, Resistor_SMD:R_1206_3216Metric_Pad1.30x1.75mm_HandSolder, F.Cu at (677.3, 306.2)
- added S11: 2MS1T2B3M2QES, Samacsys:2MS1T2B3M2QES, F.Cu at (668.1, 276.3)
- added S12: 2MS1T2B3M2QES, Samacsys:2MS1T2B3M2QES, F.Cu at (680.1, 276.3)
- added S13: 2MS1T2B3M2QES, Samacsys:2MS1T2B3M2QES, F.Cu at (654.8, 276.3)
- added S14: B3FS-4055P, Samacsys:B3FS4055P, F.Cu at (689.2, 302.6)
- added VR1: M61P104KT20T607, Samacsys:M61P104KT20T607, F.Cu at (695.8, 278.4)
- added Y1: 8MHz, Crystal:Crystal_SMD_HC49-SD_HandSoldering, F.Cu at (688.5, 314.0)
- J11, J13, J16, J19, J21, J23, J9: moved to B.Cu
- moved IC264 447.4 mm to (686.0, 364.1), turned to 90 degrees
- moved IC265 438.0 mm to (685.0, 371.5), turned to 90 degrees
- moved J15 308.7 mm to (388.9, 540.5)
- moved J16 294.1 mm to (388.9, 540.5), turned to 180 degrees
- moved J17 289.2 mm to (365.7, 540.5)
- moved U1 170.6 mm to (619.0, 279.5), turned to 0 degrees
- moved J9 167.3 mm to (320.4, 177.7)
- moved J8 160.9 mm to (320.6, 177.7), turned to 180 degrees
- moved J22 154.5 mm to (612.3, 430.2), turned to 90 degrees
- moved C1 142.4 mm to (625.2, 309.3), turned to 90 degrees
- moved J11 141.0 mm to (372.1, 181.2)
- moved C3 139.1 mm to (628.7, 309.3), turned to 90 degrees
- moved J12 136.9 mm to (398.2, 181.3), turned to 180 degrees
- moved L1 136.3 mm to (637.4, 313.3), turned to 90 degrees
- moved J10 130.3 mm to (372.1, 181.2), turned to 180 degrees
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Connections:
- J24 pad 1: /GNDA -> /DATtoADR/~{CLKd}
- J24 pad 2: /GNDA -> /ProgrammeCounter/~{CLK}
- J24 pad 3: Net-(IC1-VIN) -> /DATtoADR/LD
- J24 pad 4: Net-(IC1-VIN) -> /GNDA
- J24 pad 5: /DATtoADR/~{CLKd} -> /GNDA
- J24 pad 6: /ProgrammeCounter/~{CLK} -> Net-(IC1-VIN)
- J24 pad 7: /DATtoADR/LD -> Net-(IC1-VIN)
- J7 pad 1: /GND -> /~{CLKd}
- J7 pad 2: /GND -> /~{CLK}
- J7 pad 3: /VBUS -> /LDADR_{dis}
- J7 pad 4: /VBUS -> /GND
- J7 pad 5: /~{CLKd} -> /GND
- J7 pad 6: /~{CLK} -> /VBUS
- J7 pad 7: /LDADR_{dis} -> /VBUS
Routing:
- net /GNDA: track 0.01 -> 259.4 mm, vias 0 -> 192
- net /VCCA: track 0.02 -> 235.3 mm, vias 0 -> 113
- net /DATtoADR/LD: track 0.00 -> 178.5 mm, vias 0 -> 2
- net /DATtoADR/~{CLKd}: track 0.00 -> 147.4 mm, vias 0 -> 2
- net /ProgrammeCounter/~{CLK}: track 0.00 -> 117.9 mm, vias 0 -> 3
- net /ProgrammeCounter/~{CLR}: track 0.00 -> 108.1 mm, vias 0 -> 5
- net /CMDA4: track 0.00 -> 105.0 mm, vias 0 -> 5
- net /ADRA15: track 0.00 -> 104.9 mm, vias 0 -> 1
- net /CMDA3: track 0.00 -> 104.5 mm, vias 0 -> 5
- net /ADRA14: track 0.00 -> 102.2 mm, vias 0 -> 1
- net /ADRA13: track 0.00 -> 101.3 mm, vias 0 -> 1
- net /ADRA12: track 0.00 -> 100.1 mm, vias 0 -> 1
- net /CMDA2: track 0.00 -> 99.9 mm, vias 0 -> 5
- net /CMDA5: track 0.00 -> 99.8 mm, vias 0 -> 5
- net /CMDA1: track 0.00 -> 96.5 mm, vias 0 -> 5
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- added copper zone on In1.Cu, net /GNDA
- added copper zone on In2.Cu, net /VCCA
- added copper zone on In2.Cu, net Net-(IC1-VIN)
Other:
- board size 633.2 x 616.8 mm -> 539 x 588.5 mm
