File: 8Bit Computer ver2.0/Kicad/Computer/ProgrammeCounter.kicad_sch (KiCad schematic)
At the start: 36 parts, among them IC155 SN74F521DWR, IC156 SN74F521DWR, IC157 SN74LVC1G14DBVR, IC158 SN74LVC1G14DBVR, IC159 SN74LVC1G14DBVR, IC160 SN74LVC1G08DBVR, IC161 SN74LVC1G32DBVR, IC162 SN74HCS4075DR, IC163 SN74LVC1G32DBVR, IC164 SN74LVC1G14DBVR, IC165 CY74FCT163CTSOC, IC166 CY74FCT163CTSOC, IC167 CY74FCT163CTSOC, IC168 CY74FCT163CTSOC, IC264 SN74AHC74DR

Commit message: Fixed some Design bugs
added some pdfs
Other:
- moved on the sheet: R20, S1
Changed lines of the file:
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@@
 	(text "CLEAR Button"
 		(exclude_from_sim no)
-		(at 54.102 154.178 0)
+		(at 101.092 150.368 0)
 		(effects
 			(font
@@
 	)
 	(junction
-		(at 36.83 170.18)
+		(at 83.82 166.37)
 		(diameter 0)
 		(color 0 0 0 0)
@@
 	)
 	(junction
-		(at 106.68 167.64)
+		(at 128.27 163.83)
 		(diameter 0)
 		(color 0 0 0 0)
@@
 	)
 	(junction
-		(at 72.39 167.64)
+		(at 119.38 163.83)
 		(diameter 0)
 		(color 0 0 0 0)
@@
 	(wire
 		(pts
-			(xy 36.83 167.64) (xy 36.83 158.75)
+			(xy 83.82 163.83) (xy 83.82 154.94)
 		)
 		(stroke
@@
 	(wire
 		(pts
-			(xy 72.39 167.64) (xy 69.85 167.64)
+			(xy 119.38 163.83) (xy 116.84 163.83)
 		)
 		(stroke
@@
 	(wire
 		(pts
-			(xy 72.39 170.18) (xy 72.39 176.53)
+			(xy 119.38 166.37) (xy 119.38 172.72)
 		)
 		(stroke
@@
 	(wire
 		(pts
-			(xy 36.83 176.53) (xy 36.83 170.18)
+			(xy 83.82 172.72) (xy 83.82 166.37)
 		)
 		(stroke
@@
 	(wire
 		(pts
-			(xy 36.83 167.64) (xy 39.37 167.64)
+			(xy 83.82 163.83) (xy 86.36 163.83)
 		)
 		(stroke
@@
 	(wire
 		(pts
-			(xy 36.83 170.18) (xy 39.37 170.18)
+			(xy 83.82 166.37) (xy 86.36 166.37)
 		)
 		(stroke
@@
 	(wire
 		(pts
-			(xy 130.81 167.64) (xy 106.68 167.64)
+			(xy 135.89 163.83) (xy 128.27 163.83)
 		)
 		(stroke
@@
 	(wire
 		(pts
-			(xy 106.68 181.61) (xy 106.68 179.07)
+			(xy 128.27 177.8) (xy 128.27 175.26)
 		)
 		(stroke
@@
 	(wire
 		(pts
-			(xy 72.39 176.53) (xy 36.83 176.53)
+			(xy 119.38 172.72) (xy 83.82 172.72)
 		)
 		(stroke
@@
 	(wire
 		(pts
-			(xy 106.68 167.64) (xy 106.68 171.45)
+			(xy 128.27 163.83) (xy 128.27 167.64)
 		)
 		(stroke
@@
 	(wire
 		(pts
-			(xy 72.39 158.75) (xy 72.39 167.64)
+			(xy 119.38 154.94) (xy 119.38 163.83)
 		)
 		(stroke
@@
 	(wire
 		(pts
-			(xy 30.48 170.18) (xy 36.83 170.18)
+			(xy 77.47 166.37) (xy 83.82 166.37)
 		)
 		(stroke
@@
 	(wire
 		(pts
-			(xy 69.85 170.18) (xy 72.39 170.18)
+			(xy 116.84 166.37) (xy 119.38 166.37)
 		)
 		(stroke
@@
 	(wire
 		(pts
-			(xy 106.68 167.64) (xy 72.39 167.64)
+			(xy 128.27 163.83) (xy 119.38 163.83)
 		)
 		(stroke
@@
 	(wire
 		(pts
-			(xy 36.83 158.75) (xy 72.39 158.75)
+			(xy 83.82 154.94) (xy 119.38 154.94)
 		)
 		(stroke
@@
 	)
 	(label "~{CLR}"
-		(at 130.81 167.64 0)
+		(at 135.89 163.83 0)
 		(effects
 			(font
@@
 	)
 	(label "GND"
-		(at 30.48 170.18 180)
+		(at 77.47 166.37 180)
 		(effects
 			(font
@@
 	)
 	(label "VCC"
-		(at 106.68 181.61 270)
+		(at 128.27 177.8 270)
 		(effects
 			(font
@@
 	(symbol
 		(lib_id "Samacsys:B3FS-4055P")
-		(at 39.37 167.64 0)
+		(at 86.36 163.83 0)
 		(unit 1)
 		(exclude_from_sim no)
@@
 		(fields_autoplaced yes)
 		(property "Reference" "S1"
-			(at 54.61 160.02 0)
+			(at 101.6 156.21 0)
 			(effects
 				(font
@@
 		)
 		(property "Value" "B3FS-4055P"
-			(at 54.61 162.56 0)
+			(at 101.6 158.75 0)
 			(effects
 				(font
@@
 		)
 		(property "Footprint" "Samacsys:B3FS4055P"
-			(at 66.04 262.56 0)
+			(at 113.03 258.75 0)
 			(effects
 				(font
@@
 		)
 		(property "Datasheet" "https://omronfs.omron.com/en_US/ecb/products/pdf/en-b3fs_4.pdf"
-			(at 66.04 362.56 0)
+			(at 113.03 358.75 0)
 			(effects
 				(font
@@
 		)
 		(property "Description" "Switch Tactile N.O. SPST Projected Plunger Gull Wing 0.05A 24VDC 2.55N SMD T/R"
-			(at 39.37 167.64 0)
+			(at 86.36 163.83 0)
 			(effects
 				(font
@@
 		)
 		(property "Height" "7.3"
-			(at 66.04 562.56 0)
+			(at 113.03 558.75 0)
 			(effects
 				(font
@@
 		)
 		(property "Mouser Part Number" "653-B3FS-4055P"
-			(at 66.04 662.56 0)
+			(at 113.03 658.75 0)
 			(effects
 				(font
@@
 		)
 		(property "Mouser Price/Stock" "https://www.mouser.co.uk/ProductDetail/Omron-Electronics/B3FS-4055P?qs=8Kz9Wu9QwqWEoBxnkyUN7A%3D%3D"
-			(at 66.04 762.56 0)
+			(at 113.03 758.75 0)
 			(effects
 				(font
@@
 		)
 		(property "Manufacturer_Name" "OMRON Electronics"
-			(at 66.04 862.56 0)
+			(at 113.03 858.75 0)
 			(effects
 				(font
@@
 		)
 		(property "Manufacturer_Part_Number" "B3FS-4055P"
-			(at 66.04 962.56 0)
+			(at 113.03 958.75 0)
 			(effects
 				(font
@@
 	(symbol
 		(lib_id "Device:R")
-		(at 106.68 175.26 0)
+		(at 128.27 171.45 0)
 		(unit 1)
 		(exclude_from_sim no)
@@
 		(fields_autoplaced yes)
 		(property "Reference" "R20"
-			(at 109.22 173.9899 0)
+			(at 130.81 170.1799 0)
 			(effects
 				(font
@@
 		)
 		(property "Value" "4.7k"
-			(at 109.22 176.5299 0)
+			(at 130.81 172.7199 0)
 			(effects
 				(font
@@
 		)
 		(property "Footprint" "Resistor_SMD:R_1206_3216Metric_Pad1.30x1.75mm_HandSolder"
-			(at 104.902 175.26 90)
+			(at 126.492 171.45 90)
 			(effects
 				(font
@@
 		)
 		(property "Datasheet" "~"
-			(at 106.68 175.26 0)
+			(at 128.27 171.45 0)
 			(effects
 				(font
@@
 		)
 		(property "Description" "Resistor"
-			(at 106.68 175.26 0)
+			(at 128.27 171.45 0)
 			(effects
 				(font
