File: 8Bit Computer ver2.0/Kicad/Computer/ADR_Flash.kicad_sch (KiCad schematic)
At the start: 11 parts, among them IC203 SN74ABT245BDWR, IC204 SN74ABT245BDWR, IC206 SN74ABT245BDWR, IC207 M29F800FT55N3E2, IC210 SN74ABT245BDWR, IC211 SN74ABT245BDWR, IC214 SN74ABT245BDWR, IC215 SN74ABT245BDWR, J36 Conn_02x25_Odd_Even

Commit message: changed page numbers, every schematic is now A4
Other:
- title: (none) -> ${SHEETNAME}
Changed lines of the file:
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@@
 	(generator_version "9.0")
 	(paper "A4")
+	(title_block
+		(title "${SHEETNAME}")
+		(date "2026-03-21")
+		(rev "2.7")
+	)
 	(text "ADR Flash Program port"
 		(exclude_from_sim no)
