File: 8Bit Computer ver2.0/Kicad/Computer/ALU_Memory_Module.kicad_sch (KiCad schematic)
At the start: 7 parts, among them J10 M20-7910842R, J11 M20-7910842R, J12 M20-7910842R, J13 M20-7910842R, J14 M20-7910842R, J8 M20-7910842R, J9 M20-7910842R

Commit message: changed page numbers, every schematic is now A4
Other:
- title: (none) -> ${SHEETNAME}
Changed lines of the file:
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@@
 	(generator_version "9.0")
 	(paper "A4")
+	(title_block
+		(title "${SHEETNAME}")
+		(date "2026-03-21")
+		(rev "2.7")
+	)
 	(junction
 		(at 123.19 181.61)
