File: 8Bit Computer ver2.0/Kicad/Computer/AdderSubstractor_ALU.kicad_sch (KiCad schematic)
At the start: 15 parts, among them IC36 SN74F521DWR, IC37 SN74F521DWR, IC38 SN74F521DWR, IC50 SN74LVC1G14DBVR, IC51 SN74LVC1G14DBVR, IC52 SN74LVC1G14DBVR

Commit message: changed page numbers, every schematic is now A4
Other:
- title: (none) -> ${SHEETNAME}
Changed lines of the file:
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@@
 	(generator_version "9.0")
 	(paper "A4")
+	(title_block
+		(title "${SHEETNAME}")
+		(date "2026-03-21")
+		(rev "2.7")
+	)
 	(text "0x08\n\n"
 		(exclude_from_sim no)
