File: 8Bit Computer ver2.0/Kicad/Computer/BarrelShiftRegister.kicad_sch (KiCad schematic)
At the start: 14 parts, among them IC169 SN74LVC1G14DBVR, IC170 SN74LVC1G32DBVR, IC171 SN74AHC157DR, IC172 SN74AHC157DR, IC173 SN74AHC74DR, IC174 SN74LVC1G08DBVR, IC175 SN74AHC157DR, IC176 SN74AHC157DR, IC177 SN74LVC1G08DBVR, IC178 SN74LVC1G08DBVR, IC179 SN74AHC08DR, IC180 SN74AHC157DR, IC181 SN74AHC157DR, IC182 SN74ABT574ADWR

Commit message: changed page numbers, every schematic is now A4
Other:
- title: (none) -> ${SHEETNAME}
Changed lines of the file:
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@@
 	(generator_version "9.0")
 	(paper "A4")
+	(title_block
+		(title "${SHEETNAME}")
+		(date "2026-03-21")
+		(rev "2.7")
+	)
 	(junction
 		(at 111.76 173.99)
