File: 8Bit Computer ver2.0/Kicad/Computer/BarrelShifter.kicad_sch (KiCad schematic)
At the start: 24 parts, among them IC44 SN74F521DWR, IC45 SN74F521DWR, IC46 SN74F521DWR, IC47 SN74F521DWR, IC48 SN74LVC1G14DBVR, IC49 SN74LVC1G14DBVR, IC54 SN74LVC1G14DBVR, IC55 SN74LVC1G14DBVR, IC64 SN74LVC1G14DBVR, IC65 SN74ABT574ADWR, IC66 SN74AHC74DR, IC67 SN74LVC1G08DBVR, IC68 SN74ABT245BDWR

Commit message: changed page numbers, every schematic is now A4
Other:
- title: (none) -> ${SHEETNAME}
Changed lines of the file:
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@@
 	(generator_version "9.0")
 	(paper "A4")
+	(title_block
+		(title "${SHEETNAME}")
+		(date "2026-03-21")
+		(rev "2.7")
+	)
 	(text "0x23\n\n\n"
 		(exclude_from_sim no)
