File: 8Bit Computer ver2.0/Kicad/Computer/BinaryAND.kicad_sch (KiCad schematic)
At the start: 4 parts, among them IC89 SN74LVC1G14DBVR, IC90 SN74LVC1G08DBVR, IC91 SN74AHC74DR, IC92 SN74ABT574ADWR

Commit message: changed page numbers, every schematic is now A4
Other:
- title: (none) -> ${SHEETNAME}
Changed lines of the file:
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@@
 	(generator_version "9.0")
 	(paper "A4")
+	(title_block
+		(title "${SHEETNAME}")
+		(date "2026-03-21")
+		(rev "2.7")
+	)
 	(junction
 		(at 163.83 85.09)
