File: 8Bit Computer ver2.0/Kicad/Computer/BinaryNOT.kicad_sch (KiCad schematic)
At the start: 4 parts, among them IC93 SN74LVC1G14DBVR, IC94 SN74LVC1G14DBVR, IC95 SN74AHC74DR, IC96 SN74ABT574ADWR

Commit message: changed page numbers, every schematic is now A4
Other:
- title: (none) -> ${SHEETNAME}
Changed lines of the file:
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@@
 	(generator_version "9.0")
 	(paper "A4")
+	(title_block
+		(title "${SHEETNAME}")
+		(date "2026-03-21")
+		(rev "2.7")
+	)
 	(junction
 		(at 182.88 97.79)
