File: 8Bit Computer ver2.0/Kicad/Computer/Binary_ALU.kicad_sch (KiCad schematic)
At the start: 20 parts, among them IC69 SN74F521DWR, IC70 SN74F521DWR, IC71 SN74F521DWR, IC72 SN74F521DWR, IC77 SN74LVC1G14DBVR, IC78 SN74LVC1G14DBVR, IC79 SN74LVC1G14DBVR, IC80 SN74LVC1G14DBVR

Commit message: changed page numbers, every schematic is now A4
Other:
- title: (none) -> ${SHEETNAME}
Changed lines of the file:
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@@
 	(generator_version "9.0")
 	(paper "A4")
+	(title_block
+		(title "${SHEETNAME}")
+		(date "2026-03-21")
+		(rev "2.7")
+	)
 	(text "and"
 		(exclude_from_sim no)
