File: 8Bit Computer ver2.0/Kicad/Computer/Bitwise_ALU.kicad_sch (KiCad schematic)
At the start: 20 parts, among them IC73 SN74F521DWR, IC74 SN74F521DWR, IC75 SN74F521DWR, IC76 SN74F521DWR, IC81 SN74LVC1G14DBVR, IC82 SN74LVC1G14DBVR, IC83 SN74LVC1G14DBVR, IC84 SN74LVC1G14DBVR

Commit message: changed page numbers, every schematic is now A4
Other:
- title: (none) -> ${SHEETNAME}
Changed lines of the file:
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@@
 	(generator_version "9.0")
 	(paper "A4")
+	(title_block
+		(title "${SHEETNAME}")
+		(date "2026-03-21")
+		(rev "2.7")
+	)
 	(text "bor"
 		(exclude_from_sim no)
