File: 8Bit Computer ver2.0/Kicad/Computer/Bitwise_Binary_ALU.kicad_sch (KiCad schematic)
At the start: 4 parts, among them IC85 SN74HCS4075DR, IC86 SN74LVC1G32DBVR, IC87 SN74HCS4075DR, IC88 SN74LVC1G32DBVR

Commit message: changed page numbers, every schematic is now A4
Other:
- title: (none) -> ${SHEETNAME}
Changed lines of the file:
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@@
 	(generator_version "9.0")
 	(paper "A4")
+	(title_block
+		(title "${SHEETNAME}")
+		(date "2026-03-21")
+		(rev "2.7")
+	)
 	(bus_entry
 		(at 147.32 151.13)
