File: 8Bit Computer ver2.0/Kicad/Computer/CMD_DAT_Flash.kicad_sch (KiCad schematic)
At the start: 13 parts, among them IC198 DS1100Z-20+, IC199 SN74AHC74DR, IC200 SN74ABT245BDWR, IC201 SN74ABT245BDWR, IC202 SN74ABT245BDWR, IC205 M29F800FT55N3E2, IC208 SN74ABT245BDWR, IC209 SN74ABT245BDWR, IC212 SN74ABT245BDWR, IC213 SN74ABT245BDWR, J35 Conn_02x25_Odd_Even

Commit message: changed page numbers, every schematic is now A4
Other:
- title: (none) -> ${SHEETNAME}
Changed lines of the file:
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@@
 	(generator_version "9.0")
 	(paper "A4")
+	(title_block
+		(title "${SHEETNAME}")
+		(date "2026-03-21")
+		(rev "2.7")
+	)
 	(text "DATA and CMD Flash Program port"
 		(exclude_from_sim no)
