File: 8Bit Computer ver2.0/Kicad/Computer/Capacitors_ALU.kicad_sch (KiCad schematic)
At the start: 187 parts

Commit message: changed page numbers, every schematic is now A4
Other:
- title: (none) -> ${SHEETNAME}
Changed lines of the file:
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@@
 	(generator_version "9.0")
 	(paper "A4")
+	(title_block
+		(title "${SHEETNAME}")
+		(date "2026-03-21")
+		(rev "2.7")
+	)
 	(junction
 		(at 255.27 77.47)
