File: 8Bit Computer ver2.0/Kicad/Computer/Clocks_Control_Module.kicad_sch (KiCad schematic)
At the start: 33 parts, among them IC266 SN74LVC1GU04DCKR, IC267 TMUX1309DYYR, IC268 SN74LVC1G14DBVR, IC269 LM555CMX_NOPB, IC270 SN74AHC74DR, Y1 4MHz

Commit message: changed page numbers, every schematic is now A4
Other:
- title: (none) -> ${SHEETNAME}
Changed lines of the file:
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@@
 	(generator_version "9.0")
 	(paper "A4")
+	(title_block
+		(title "${SHEETNAME}")
+		(date "2026-03-21")
+		(rev "2.7")
+	)
 	(text "Pierce Oscillator"
 		(exclude_from_sim no)
