File: 8Bit Computer ver2.0/Kicad/Computer/Comparator_ALU.kicad_sch (KiCad schematic)
At the start: 15 parts, among them IC41 SN74F521DWR, IC42 SN74F521DWR, IC43 SN74F521DWR, IC61 SN74LVC1G14DBVR, IC62 SN74LVC1G14DBVR, IC63 SN74LVC1G14DBVR

Commit message: changed page numbers, every schematic is now A4
Other:
- title: (none) -> ${SHEETNAME}
Changed lines of the file:
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@@
 	(generator_version "9.0")
 	(paper "A4")
+	(title_block
+		(title "${SHEETNAME}")
+		(date "2026-03-21")
+		(rev "2.7")
+	)
 	(text "0x15\n\n"
 		(exclude_from_sim no)
