File: 8Bit Computer ver2.0/Kicad/Computer/Control_Module.kicad_sch (KiCad schematic)
At the start: 27 parts, among them IC1 MP2338GTL-Z, IC238 SN74LVC1G14DBVR, IC3 DS1100Z-150+, J18 M20-8890845, J19 M20-8890845, J20 M20-8890845, J21 M20-8890845, J22 M20-8890845, J23 M20-8890845, J24 M20-8890845

Commit message: changed page numbers, every schematic is now A4
Other:
- title: (none) -> ${SHEETNAME}
Changed lines of the file:
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@@
 	(generator_version "9.0")
 	(paper "A4")
+	(title_block
+		(title "${SHEETNAME}")
+		(date "2026-03-21")
+		(rev "2.7")
+	)
 	(text "90ns"
 		(exclude_from_sim no)
@@
 			(project "Computer"
 				(path "/1196a00e-6878-4d6d-82b7-9e052dfe7c14/4a034013-5cf2-4646-a922-b4f8e2c339f0"
-					(page "30")
+					(page "31")
 				)
 			)
@@
 			(project "Computer"
 				(path "/1196a00e-6878-4d6d-82b7-9e052dfe7c14/4a034013-5cf2-4646-a922-b4f8e2c339f0"
-					(page "32")
+					(page "33")
 				)
 			)
@@
 			(project "Computer"
 				(path "/1196a00e-6878-4d6d-82b7-9e052dfe7c14/4a034013-5cf2-4646-a922-b4f8e2c339f0"
-					(page "31")
+					(page "32")
 				)
 			)
