File: 8Bit Computer ver2.0/Kicad/Computer/FlagRegister_ALU.kicad_sch (KiCad schematic)
At the start: 23 parts, among them IC32 SN74F521DWR, IC33 SN74F521DWR, IC34 SN74F521DWR, IC35 SN74F521DWR, IC57 SN74LVC1G14DBVR, IC58 SN74LVC1G14DBVR, IC59 SN74LVC1G14DBVR, IC60 SN74LVC1G14DBVR

Commit message: changed page numbers, every schematic is now A4
Other:
- title: (none) -> ${SHEETNAME}
Changed lines of the file:
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@@
 	(generator_version "9.0")
 	(paper "A4")
+	(title_block
+		(title "${SHEETNAME}")
+		(date "2026-03-21")
+		(rev "2.7")
+	)
 	(text "0010 0001"
 		(exclude_from_sim no)
