File: 8Bit Computer ver2.0/Kicad/Computer/RAM.kicad_sch (KiCad schematic)
At the start: 11 parts, among them IC216 SN74F521DWR, IC217 SN74F521DWR, IC218 SN74LVC1G14DBVR, IC219 SN74LVC1G14DBVR, IC220 SN74LVC1G14DBVR, IC221 SN74AHC74DR, IC222 SN74LVC1G08DBVR, IC223 AS7C1024B-12TCN, IC282 SN74LVC1G14DBVR, IC283 SN74HCS32DR

Commit message: changed page numbers, every schematic is now A4
Other:
- title: (none) -> ${SHEETNAME}
Changed lines of the file:
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@@
 	(generator_version "9.0")
 	(paper "A4")
+	(title_block
+		(title "${SHEETNAME}")
+		(date "2026-03-21")
+		(rev "2.7")
+	)
 	(text "Load from RAM"
 		(exclude_from_sim no)
