File: 8Bit Computer ver2.0/Kicad/Computer/Register_A.kicad_sch (KiCad schematic)
At the start: 14 parts, among them IC12 SN74LVC1G14DBVR, IC14 SN74LVC1G14DBVR, IC17 SN74LVC1G14DBVR, IC19 SN74ABT574ADWR, IC22 SN74AHC74DR, IC25 SN74LVC1G08DBVR, IC28 SN74ABT245BDWR, IC6 SN74F521DWR, IC7 SN74F521DWR

Commit message: changed page numbers, every schematic is now A4
Other:
- title: (none) -> ${SHEETNAME}
Changed lines of the file:
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@@
 	(generator_version "9.0")
 	(paper "A4")
+	(title_block
+		(title "${SHEETNAME}")
+		(date "2026-03-21")
+		(rev "2.7")
+	)
 	(text "0x18"
 		(exclude_from_sim no)
