File: 8Bit Computer ver2.0/Kicad/Computer/Register_B.kicad_sch (KiCad schematic)
At the start: 14 parts, among them IC13 SN74LVC1G14DBVR, IC16 SN74LVC1G14DBVR, IC18 SN74LVC1G14DBVR, IC20 SN74ABT574ADWR, IC23 SN74AHC74DR, IC26 SN74LVC1G08DBVR, IC29 SN74ABT245BDWR, IC8 SN74F521DWR, IC9 SN74F521DWR

Commit message: changed page numbers, every schematic is now A4
Other:
- title: (none) -> ${SHEETNAME}
Changed lines of the file:
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@@
 	(generator_version "9.0")
 	(paper "A4")
+	(title_block
+		(title "${SHEETNAME}")
+		(date "2026-03-21")
+		(rev "2.7")
+	)
 	(text "REGISTER B\n\n"
 		(exclude_from_sim no)
